File: kicad/nanomount.kicad_pcb (KiCad board)
At the start: 2 copper layers, 45.7 x 43.1 mm, 2 parts, among them J1 CONN_02X13, U1 ArduinoNano

Commit message: changes in kicad design
Other:
- board size 45.7 x 43.1 mm -> 50.8 x 45.7 mm
Changed lines of the file:
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@@
-(kicad_pcb (version 20170123) (host pcbnew "(2017-06-02 revision ac9a64a17)-master")
+(kicad_pcb (version 20170123) (host pcbnew "(2017-06-11 revision 44b118f8c)-makepkg")
   (general
     (links 18)
     (no_connects 2)
-    (area 124.384999 87.745 179.370001 134.620001)
+    (area 121.844999 87.745 181.910001 137.235001)
     (thickness 1.6)
-    (drawings 13)
+    (drawings 10)
     (tracks 83)
     (zones 0)
@@
       (net 26 THEL))
   )
-  (dimension 43.18 (width 0.3) (layer B.SilkS)
-    (gr_text "43.180 mm" (at 172.72 113.03 270) (layer B.SilkS)
+  (dimension 45.72 (width 0.3) (layer F.SilkS)
+    (gr_text "45.720 mm" (at 175.26 114.3 270) (layer F.SilkS)
       (effects (font (size 1.5 1.5) (thickness 0.3)))
     )
-    (feature1 (pts (xy 172.72 134.62) (xy 172.72 134.62)))
-    (feature2 (pts (xy 172.72 91.44) (xy 172.72 91.44)))
-    (crossbar (pts (xy 172.72 91.44) (xy 172.72 134.62)))
-    (arrow1a (pts (xy 172.72 134.62) (xy 172.133579 133.493496)))
-    (arrow1b (pts (xy 172.72 134.62) (xy 173.306421 133.493496)))
-    (arrow2a (pts (xy 172.72 91.44) (xy 172.133579 92.566504)))
-    (arrow2b (pts (xy 172.72 91.44) (xy 173.306421 92.566504)))
-  )
-  (dimension 45.72 (width 0.3) (layer B.SilkS)
-    (gr_text "45.720 mm" (at 147.32 88.9) (layer B.SilkS)
+    (feature1 (pts (xy 175.26 137.16) (xy 175.26 137.16)))
+    (feature2 (pts (xy 175.26 91.44) (xy 175.26 91.44)))
+    (crossbar (pts (xy 175.26 91.44) (xy 175.26 137.16)))
+    (arrow1a (pts (xy 175.26 137.16) (xy 174.673579 136.033496)))
+    (arrow1b (pts (xy 175.26 137.16) (xy 175.846421 136.033496)))
+    (arrow2a (pts (xy 175.26 91.44) (xy 174.673579 92.566504)))
+    (arrow2b (pts (xy 175.26 91.44) (xy 175.846421 92.566504)))
+  )
+  (dimension 50.8 (width 0.3) (layer F.SilkS)
+    (gr_text "50.800 mm" (at 147.32 88.9) (layer F.SilkS)
       (effects (font (size 1.5 1.5) (thickness 0.3)))
     )
-    (feature1 (pts (xy 170.18 88.9) (xy 170.18 88.9)))
-    (feature2 (pts (xy 124.46 88.9) (xy 124.46 88.9)))
-    (crossbar (pts (xy 124.46 88.9) (xy 170.18 88.9)))
-    (arrow1a (pts (xy 170.18 88.9) (xy 169.053496 89.486421)))
-    (arrow1b (pts (xy 170.18 88.9) (xy 169.053496 88.313579)))
-    (arrow2a (pts (xy 124.46 88.9) (xy 125.586504 89.486421)))
-    (arrow2b (pts (xy 124.46 88.9) (xy 125.586504 88.313579)))
-  )
-  (gr_line (start 170.18 91.44) (end 170.18 93.98) (layer Edge.Cuts) (width 0.15))
-  (gr_line (start 124.46 91.44) (end 170.18 91.44) (layer Edge.Cuts) (width 0.15))
-  (gr_line (start 124.46 93.98) (end 124.46 91.44) (layer Edge.Cuts) (width 0.15))
+    (feature1 (pts (xy 121.92 88.9) (xy 121.92 88.9)))
+    (feature2 (pts (xy 172.72 88.9) (xy 172.72 88.9)))
+    (crossbar (pts (xy 172.72 88.9) (xy 121.92 88.9)))
+    (arrow1a (pts (xy 121.92 88.9) (xy 123.046504 88.313579)))
+    (arrow1b (pts (xy 121.92 88.9) (xy 123.046504 89.486421)))
+    (arrow2a (pts (xy 172.72 88.9) (xy 171.593496 88.313579)))
+    (arrow2b (pts (xy 172.72 88.9) (xy 171.593496 89.486421)))
+  )
+  (gr_line (start 121.92 91.44) (end 172.72 91.44) (layer Edge.Cuts) (width 0.15))
   (gr_text PWMAZv (at 150.622 94.107) (layer B.Cu)
     (effects (font (size 1.5 1.5) (thickness 0.3)) (justify mirror))
@@
     (effects (font (size 1.5 1.5) (thickness 0.3)) (justify mirror))
   )
-  (gr_line (start 170.18 134.493) (end 170.18 93.98) (layer Edge.Cuts) (width 0.15))
-  (gr_line (start 124.46 134.493) (end 170.18 134.493) (layer Edge.Cuts) (width 0.15))
-  (gr_line (start 124.46 132.08) (end 124.46 134.493) (layer Edge.Cuts) (width 0.15))
-  (gr_line (start 124.46 93.98) (end 124.46 132.08) (layer Edge.Cuts) (width 0.15))
+  (gr_line (start 172.72 137.16) (end 172.72 91.44) (layer Edge.Cuts) (width 0.15))
+  (gr_line (start 121.92 137.16) (end 172.72 137.16) (layer Edge.Cuts) (width 0.15))
+  (gr_line (start 121.92 91.44) (end 121.92 137.16) (layer Edge.Cuts) (width 0.15))
   (segment (start 162.052 101.854) (end 162.052 109.014238) (width 0.5) (layer B.Cu) (net 2))
   (segment (start 162.052 109.014238) (end 165.850001 112.812239) (width 0.5) (layer B.Cu) (net 2))
